File: ASIC.kicad_sch (KiCad schematic)
At the start: 66 parts, among them U10 BM1370_mode1, U11 MCP1824T-1202E/OT, U12 MCP1824T-0802E, U2 SN74AVC4T774, U8 25MHz, U9 BM1370_mode1

Commit message: add LCSC code
Parts:
- C38, C54, C55, C56, C57, C58, C59, C60, C61, C62: LCSC (none) -> C344022
- C51, C52, C53: LCSC (none) -> C5137487
- C64, C65, C66, C67, C68, C69, C70, C71, C72, C73, C74, C75, C76, C77, C78, C79, C80, C81, C82, C83, C84, C85, C86, C87, C88, C89, C90, C91: LCSC (none) -> C181017
- R23: LCSC (none) -> C93942
- R24: LCSC (none) -> C60489
- R26, R28: LCSC (none) -> C106235
- R27: LCSC (none) -> C852711

Commit message: final update
Parts:
- U10, U9: LCSC (none) -> C9900140670
- U11: value MCP1824T-1202E/OT -> RT9080-12GJ5; DK MCP1824T-1202E/OTCT-ND -> RT9080-12GJ5; LCSC (none) -> C2983593
- U12: value MCP1824T-0802E -> RT9080-08GJ5-MS; DK MCP1824T-0802E/OTCT-ND -> (none); LCSC (none) -> C30602453
- U2: value SN74AVC4T774 -> SN74AXC4T774BQBR; LCSC (none) -> C2862903
Changed lines of the file:
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@@
 			)
 		)
+		(property "LCSC" "C9900140670"
+			(at 99.06 114.3 0)
+			(effects
+				(font
+					(size 1.27 1.27)
+				)
+			)
+		)
 		(pin "11"
 		)
@@
 			)
 		)
-		(property "Value" "MCP1824T-1202E/OT"
+		(property "Value" "RT9080-12GJ5"
 			(at 61.468 167.386 0)
 			(effects
@@
 			)
 		)
-		(property "DK" "MCP1824T-1202E/OTCT-ND"
+		(property "DK" "RT9080-12GJ5"
 			(at 60.96 172.72 0)
 			(effects
@@
 			)
 		)
+		(property "LCSC" "C2983593"
+			(at 60.96 172.72 0)
+			(effects
+				(font
+					(size 1.27 1.27)
+				)
+			)
+		)
 		(pin "3"
 		)
@@
 			)
 		)
-		(property "Value" "SN74AVC4T774"
+		(property "Value" "SN74AXC4T774BQBR"
 			(at 199.39 21.59 0)
 			(effects
@@
 			)
 		)
-		(property "LCSC" ""
+		(property "LCSC" "C2862903"
 			(at 199.39 34.29 0)
 			(effects
@@
 			)
 		)
-		(property "Value" "MCP1824T-0802E"
+		(property "Value" "RT9080-08GJ5-MS"
 			(at 130.81 167.386 0)
 			(effects
@@
 			)
 		)
-		(property "DK" "MCP1824T-0802E/OTCT-ND"
+		(property "DK" ""
 			(at 130.81 172.72 0)
 			(effects
@@
 			)
 		)
+		(property "LCSC" "C30602453"
+			(at 130.81 172.72 0)
+			(effects
+				(font
+					(size 1.27 1.27)
+				)
+			)
+		)
 		(pin "3"
 		)
@@
 			)
 		)
+		(property "LCSC" "C9900140670"
+			(at 203.2 114.3 0)
+			(effects
+				(font
+					(size 1.27 1.27)
+				)
+			)
+		)
