File: ESP32.kicad_sch (KiCad schematic)
At the start: 18 parts, among them J2 Conn_01x08, J3 Conn_01x04, J4 USB_C_Receptacle_USB2.0, J8 TC2030-IDC, SW1 SWITCH-SPST, SW2 SWITCH-SPST, U6 ESP32-S3-WROOM-1

Commit message: add LCSC code
Parts:
- C48: LCSC (none) -> C106201
- C49: LCSC (none) -> C344022
- J4: LCSC (none) -> C2982555
- R20: LCSC (none) -> C60489
- SW1, SW2: LCSC (none) -> C7498203
- U6: LCSC (none) -> C2913202
Changed lines of the file:
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@@
+			)
+		)
+		(property "LCSC" "C7498203"
+			(at 96.52 52.07 0)
+			(effects
+				(font
+					(size 1.27 1.27)
+				)
+				(hide yes)
 			)
 		)
@@
 			)
 		)
+		(property "LCSC" "C2982555"
+			(at 257.81 66.04 0)
+			(effects
+				(font
+					(size 1.27 1.27)
+				)
+				(hide yes)
+			)
+		)
 		(pin "B7"
 		)
@@
 					(size 1.27 1.27)
 				)
+			)
+		)
+		(property "LCSC" "C344022"
+			(at 50.8 133.35 0)
+			(effects
+				(font
+					(size 1.27 1.27)
+				)
+				(hide yes)
 			)
 		)
@@
 			)
 		)
+		(property "LCSC" "C2913202"
+			(at 140.97 99.06 0)
+			(effects
+				(font
+					(size 1.27 1.27)
+				)
+				(hide yes)
+			)
+		)
 		(pin "3"
 		)
@@
 			)
 		)
+		(property "LCSC" "C7498203"
+			(at 57.15 52.07 0)
+			(effects
+				(font
+					(size 1.27 1.27)
+				)
+				(hide yes)
+			)
+		)
 		(pin "2"
 		)
@@
 			)
 		)
+		(property "LCSC" "C60489"
+			(at 66.04 48.26 0)
+			(effects
+				(font
+					(size 1.27 1.27)
+				)
+				(hide yes)
+			)
+		)
 		(pin "2"
 		)
@@
 			)
 		)
+		(property "LCSC" "C106201"
+			(at 66.04 58.42 0)
+			(effects
+				(font
+					(size 1.27 1.27)
+				)
+				(hide yes)
+			)
+		)

Commit message: final update
Parts:
- SW1, SW2: LCSC C7498203 -> C2886885
Changed lines of the file:
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@@
 			)
 		)
-		(property "LCSC" "C7498203"
+		(property "LCSC" "C2886885"
 			(at 96.52 52.07 0)
 			(effects
@@
 			)
 		)
-		(property "LCSC" "C7498203"
+		(property "LCSC" "C2886885"
 			(at 57.15 52.07 0)
 			(effects
